File: schematics/macropad_v0.5.kicad_sch (KiCad schematic)
At the start: 58 parts, among them SW0 SW_Push, SW1 SW_Push, SW10 SW_Push, SW11 SW_Push, SW12 SW_Push, SW13 SW_Push, SW14 SW_Push, SW15 SW_Push, SW16 SW_Push, SW17 SW_Push, SW18 SW_Push, SW19 SW_Push, SW2 SW_Push, SW20 SW_Push, SW21 SW_Push, SW3 SW_Push, SW4 SW_Push, SW5 SW_Push, SW6 SW_Push, SW7 SW_Push, SW8 SW_Push, SW9 SW_Push, U1 RP2040

Commit message: Add files via upload
Parts:
- added C12: 100nF, symbol Device:C_Small
- added C13, C14: 15pF, symbol Device:C_Small
- added C15: 100mF, symbol Device:C_Small
- added C16, C17: 10uF, Adafruit MacroPad 2040 rev D:0805-NO, symbol Device:C_Small
- added C18, C19: 1uF, Adafruit MacroPad 2040 rev D:0603-NO, symbol Device:C_Small
- added C20: .1uF, symbol Device:C_Small
- added C21, C22, C23: 10uF, symbol Device:C_Small
- added D22: PRTR5V0U2X, Package_TO_SOT_SMD:SOT-143, symbol Power_Protection:PRTR5V0U2X
- added D23, D24, D25, D26, D27, D28, D29, D30, D31, D32, D33, D34, D35, D36, D37, D38, D39, D40, D41, D42, D44, D46: SK6812MINI, LED_SMD:LED_SK6812MINI_PLCC4_3.5x3.5mm_P1.75mm, symbol LED:SK6812MINI
- added F1: 500m, symbol Device:Polyfuse_Small
- added J1: Conn_01x06, symbol Connector_Generic:Conn_01x06
- added J2: Conn_01x02, symbol Connector_Generic:Conn_01x02
- added R10: 10k, symbol Device:R_Small_US
- added R3: 10k, symbol Device:R_US
- added R4: 330, symbol Device:R_US
- added R5, R6: 5.1k, symbol Device:R_Small_US
- added R7: 1k, symbol Device:R_Small_US
- added R8: 5.1K Pack, Adafruit MacroPad 2040 rev D:RESPACK_4X0603, symbol Adafruit MacroPad 2040 rev D-eagle-import:RESISTOR_4PACK
- added R9: 680K, Adafruit MacroPad 2040 rev D:0603-NO, symbol Device:R_Small_US
- added SW22: SW_Push, symbol Switch:SW_Push
- added SW23: RotaryEncoder_Switch, symbol Device:RotaryEncoder_Switch
- added U2: W25Q128JVS, Package_SO:SOIC-8_5.23x5.23mm_P1.27mm, symbol Memory_Flash:W25Q128JVS
- added U3: RT9080-33GJ5, TSOT-23-5_RIT, symbol 2024-10-16_19-02-49:RT9080-33GJ5
- added U4: 74AHCT1G125, symbol 74xGxx:74AHCT1G125
- added USB1: HRO-TYPE-C-31-M-12, symbol Type-C:HRO-TYPE-C-31-M-12
- added X1: ABM8-272-T3, ABM8-272-T3_ABR, symbol 2024-10-07_19-23-58:ABM8-272-T3
- added X2: ZJY130-2864KSWLG22, Adafruit MacroPad 2040 rev D:ZJY130-2864KSWLG22, symbol Adafruit MacroPad 2040 rev D-eagle-import:ZJY130-2864KSWLG22
Connections:
- net GND: now also C13.1, C14.1, C15.2, C16.1, C17.1, C20.2, C21.2, C22.2, C23.2, D22.1 (GND), D23.2 (VSS), D24.2 (VSS), D25.2 (VSS), D26.2 (VSS), D27.2 (VSS), D28.2 (VSS), D29.2 (VSS), D30.2 (VSS), D31.2 (VSS), D32.2 (VSS), D33.2 (VSS), D34.2 (VSS), D35.2 (VSS), D36.2 (VSS), D37.2 (VSS), D38.2 (VSS), D39.2 (VSS), D40.2 (VSS), D41.2 (VSS), D42.2 (VSS), D44.2 (VSS), D46.2 (VSS), J1.1 (Pin_1), J2.1 (Pin_1), R10.2, R4.2, R5.2, R6.2, R8.5 (2), R9.1, SW23.C, SW23.S2, U2.4 (GND), U3.2 (GND), U4.1, U4.3 (GND), USB1.1 (GND), USB1.12 (GND), USB1.13 (SHIELD), X1.2, X1.4, X2.16 (VSS), X2.6 (VSS), X2.SUPPORT1 (VSS), X2.SUPPORT2 (VSS)
- net QSPI_SCLK: now also U2.6 (CLK)
- net QSPI_SD0: now also U2.5 (DI(IO0))
- net QSPI_SD1: now also U2.2 (DO(IO1))
- net QSPI_SD2: now also U2.3 (IO2)
- net QSPI_SD3: now also U2.7 (IO3)
- net RUN: now also C12.1, R3.1, SW22.2
- net XIN: now also C13.2, X1.1
- net XOUT: now also C14.2, X1.3
- net QSPI_SS renamed +3.3V
- net +3.3V: now also C15.1, C23.1, R3.2, R7.2, U2.1 (~{CS}), U2.8 (VCC), U3.5 (VOUT)
- new net: D36.1 (DOUT), D38.3 (DIN)
- new net: D36.3 (DIN), D37.1 (DOUT)
- new net: D27.1 (DOUT), D28.3 (DIN)
- new net: D26.1 (DOUT), D27.3 (DIN)
- new net: D24.1 (DOUT), D25.3 (DIN)
- new net: D23.1 (DOUT), D24.3 (DIN)
- new net: D42.1 (DOUT), D44.3 (DIN)
- new net: D41.1 (DOUT), D42.3 (DIN)
- new net: D33.1 (DOUT), D34.3 (DIN)
- new net: D32.1 (DOUT), D33.3 (DIN)
- new net: D25.1 (DOUT), D26.3 (DIN)
- new net: D34.1 (DOUT), D35.3 (DIN)
- new net: D44.1 (DOUT), D46.3 (DIN)
- new net: D38.1 (DOUT), D39.3 (DIN)
- new net: R6.1, USB1.4 (CC1)
- new net: R9.2, X2.13 (IREF)
- new net: D28.1 (DOUT), D29.3 (DIN)
- new net: D31.1 (DOUT), D32.3 (DIN)
- new net: D30.1 (DOUT), D31.3 (DIN)
- new net: D29.1 (DOUT), D30.3 (DIN)
- new net: D40.1 (DOUT), D41.3 (DIN)
- new net: C12.2, R4.1, SW22.1
- new net: C18.1, X2.4 (C1-)
- new net: C18.2, X2.3 (C1+)
- new net: C19.2, X2.1 (C2+)
- new net: C19.1, X2.2 (C2-)
- new net: R5.1, USB1.10 (CC2)
- new net: D35.1 (DOUT), D37.3 (DIN)
- new net: D39.1 (DOUT), D40.3 (DIN)
- new net +5V: C20.1, C21.1, C22.1, D22.4 (VCC), D23.4 (VDD), D24.4 (VDD), D25.4 (VDD), D26.4 (VDD), D27.4 (VDD), D28.4 (VDD), D29.4 (VDD), D30.4 (VDD), D31.4 (VDD), D32.4 (VDD), D33.4 (VDD), D34.4 (VDD), D35.4 (VDD), D36.4 (VDD), D37.4 (VDD), D38.4 (VDD), D39.4 (VDD), D40.4 (VDD), D41.4 (VDD), D42.4 (VDD), D44.4 (VDD), D46.4 (VDD), F1.2, J1.6 (Pin_6), U3.1 (VIN), U3.3 (EN), U4.5 (VCC)
- new net 3.3V: X2.5 (VBAT), X2.7 (VDD)
- new net D+: D22.3 (I/O2), USB1.6 (DP1), USB1.8 (DP2)
- new net D-: D22.2 (I/O1), USB1.5 (DN2), USB1.7 (DN1)
- new net GPIO?: SW23.A, SW23.B, SW23.S1
- new net MISO: J1.4 (Pin_4)
- new net MOSI: J1.3 (Pin_3), X2.12 (MOSI)
- new net NEOPIXEL: R10.1, U4.2
- new net NEOPIXEL_5V: D23.3 (DIN), U4.4
- new net OLED_CS: X2.8 (~{CS})
- new net OLED_DC: X2.10 (D/~{C})
- new net OLED_RST: R8.4 (1), X2.9 (~{RES})
- new net RST: J1.5 (Pin_5)
- new net SCK: J1.2 (Pin_2), X2.11 (SCK)
- new net USB_BOOT: J2.2 (Pin_2), R7.1
- new net VBUS: F1.1, USB1.11 (VBUS), USB1.2 (VBUS)
- new net VCC: C17.2, X2.15 (VCC)
- new net VCOMH: C16.2, X2.14 (VCOMH)
- no-connect marks 0 -> 3
Other:
- note added: "Crystal Oscillator"
- note added: "Data ESD Protection"
- note added: "Flash Memory"
- note added: "Media Controller"
- note added: "OLED Display Connection"
- note added: "Power and Filtering"
- note added: "RGB Array"
- note added: "Reset Circuit"
- note added: "SPI Header"
- note added: "USB-C Connector"
